Commit message: Add files via upload

File: 01-panda_force_control/panda_arm_FT_sensor.urdf (robot description, URDF)
Before this commit: robot panda, 8 links, 7 joints
Links:
- added link link10, mass 0.000001
- added link link11, mass 0.000001
- added link link12, mass 0.00000001
- added link link13, mass 1.5; collision sphere radius=0.05; visual sphere radius=0.05
- added link link8, mass 0.00000001
- added link link9, mass 0.00000001
- link link7: geometry visual mesh filename=../../../robot_models/Panda/meshes/link7.obj
Joints:
- added joint joint10: type prismatic, parent link9, child link10, axis 0 0 1, limit lower=-0.0175 upper=3.7525 effort=12 velocity=2.6100
- added joint joint11: type revolute, parent link10, child link11, axis 1 0 0, limit lower=-0.0175 upper=3.7525 effort=12 velocity=2.6100
- added joint joint12: type revolute, parent link11, child link12, axis 0 1 0, limit lower=-0.0175 upper=3.7525 effort=12 velocity=2.6100
- added joint joint13: type revolute, parent link12, child link13, axis 0 0 1, limit lower=-0.0175 upper=3.7525 effort=12 velocity=2.6100
- added joint joint8: type prismatic, parent link7, child link8, axis 1 0 0, limit lower=-0.0175 upper=3.7525 effort=12 velocity=2.6100
- added joint joint9: type prismatic, parent link8, child link9, axis 0 1 0, limit lower=-0.0175 upper=3.7525 effort=12 velocity=2.6100

File: 01-panda_force_control/panda_arm_force_sensor.urdf (robot description, URDF)
Before this commit: robot panda, 8 links, 7 joints
Links:
- added link link10, mass 1.5; collision sphere radius=0.05; visual sphere radius=0.05
- added link link8, mass 0.000001
- added link link9, mass 0.000001
- link link7: geometry visual mesh filename=../../../robot_models/Panda/meshes/link7.obj
Joints:
- added joint joint10: type prismatic, parent link9, child link10, axis 0 0 1, limit lower=-0.0175 upper=3.7525 effort=12 velocity=2.6100
- added joint joint8: type prismatic, parent link7, child link8, axis 1 0 0, limit lower=-0.0175 upper=3.7525 effort=12 velocity=2.6100
- added joint joint9: type prismatic, parent link8, child link9, axis 0 1 0, limit lower=-0.0175 upper=3.7525 effort=12 velocity=2.6100
