Commit message: modified inertial parameters object to match SVH hand

File: 01-panda_force_control/panda_arm.urdf (robot description, URDF)
Before this commit: robot panda, 8 links, 7 joints
Links:
- link link7: mass 1.5 -> 2.0

File: 01-panda_force_control/panda_arm_FT_sensor.urdf (robot description, URDF)
Before this commit: robot panda, 14 links, 13 joints
Links:
- link link13: mass 1.5 -> 2.0

Commit message: modified inertial params last link to match hand

File: 01-panda_force_control/panda_arm.urdf (robot description, URDF)
Before this commit: robot panda, 8 links, 7 joints
Links:
- link link7: mass 2.0 -> 1.808

File: 01-panda_force_control/panda_arm_FT_sensor.urdf (robot description, URDF)
Before this commit: robot panda, 14 links, 13 joints
Links:
- link link13: mass 2.0 -> 1.808
