Commit message: debugging estimation

File: 01-panda_force_control/06-urdf_files/panda_arm.urdf (robot description, URDF)
Before this commit: robot panda, 9 links, 8 joints
Links:
- removed link link8
- link link0: geometry 
- link link1: geometry 
- link link2: geometry 
- link link3: geometry 
- link link4: geometry 
- link link5: geometry 
- link link6: geometry 
- link link7: mass 0.5 -> 1.8; geometry 
Joints:
- removed joint joint8

File: 01-panda_force_control/06-urdf_files/panda_arm_FT_sensor.urdf (robot description, URDF)
Before this commit: robot panda, 14 links, 13 joints
Links:
- link link0: geometry 
- link link1: geometry 
- link link13: geometry collision sphere radius=0.05
- link link2: geometry 
- link link3: geometry 
- link link4: geometry 
- link link5: geometry 
- link link6: geometry 
- link link7: geometry 
Joints:
- joint joint10: origin xyz=0 0 0 rpy=0 0 0 -> (none)
- joint joint11: origin xyz=0 0 0 rpy=0 0 0 -> (none)
- joint joint12: origin xyz=0 0 0 rpy=0 0 0 -> (none)
- joint joint13: origin xyz=0 0 0 rpy=0 0 0 -> (none)
- joint joint9: origin xyz=0 0 0 rpy=0 0 0 -> (none)

Commit message: added mean filter

File: 01-panda_force_control/06-urdf_files/panda_arm.urdf (robot description, URDF)
Before this commit: robot panda, 8 links, 7 joints
Links:
- link link7: geometry visual mesh filename=../../../robot_models/Panda/meshes/link7.obj

Commit message: saving everything

File: 01-panda_force_control/06-urdf_files/panda_arm.urdf (robot description, URDF)
Before this commit: robot panda, 8 links, 7 joints
Links:
- link link0: geometry visual mesh filename=../../../robot_models/Panda/meshes/link0.obj
- link link1: geometry visual mesh filename=../../../robot_models/Panda/meshes/link1.obj
- link link2: geometry visual mesh filename=../../../robot_models/Panda/meshes/link2.obj
- link link3: geometry visual mesh filename=../../../robot_models/Panda/meshes/link3.obj
- link link4: geometry visual mesh filename=../../../robot_models/Panda/meshes/link4.obj
- link link5: geometry visual mesh filename=../../../robot_models/Panda/meshes/link5.obj
- link link6: geometry visual mesh filename=../../../robot_models/Panda/meshes/link6.obj
