Commit message: working on trajectory, adjusted virtual force sensor

File: 01-panda_force_control/06-urdf_files/panda_arm_FT_sensor.urdf (robot description, URDF)
Before this commit: robot panda-sensor, 14 links, 13 joints
Links:
- link link0: geometry visual mesh filename=../../../robot_models/Panda/meshes/link0.obj
- link link1: geometry visual mesh filename=../../../robot_models/Panda/meshes/link1.obj
- link link13: geometry collision sphere radius=0.05; visual sphere radius=0.05
- link link2: geometry visual mesh filename=../../../robot_models/Panda/meshes/link2.obj
- link link3: geometry visual mesh filename=../../../robot_models/Panda/meshes/link3.obj
- link link4: geometry visual mesh filename=../../../robot_models/Panda/meshes/link4.obj
- link link5: geometry visual mesh filename=../../../robot_models/Panda/meshes/link5.obj
- link link6: geometry visual mesh filename=../../../robot_models/Panda/meshes/link6.obj
- link link7: geometry visual mesh filename=../../../robot_models/Panda/meshes/link7.obj

Commit message: prepared examples for src files

File: 01-panda_force_control/06-urdf_files/panda_arm_FT_sensor.urdf (robot description, URDF)
Before this commit: robot panda-sensor, 14 links, 13 joints
Links:
- link link0: geometry visual mesh filename=../../../robot_models/Panda/newmeshes/link0.obj
- link link1: geometry visual mesh filename=../../../robot_models/Panda/newmeshes/link1.obj
- link link2: geometry visual mesh filename=../../../robot_models/Panda/newmeshes/link2.obj
- link link3: geometry visual mesh filename=../../../robot_models/Panda/newmeshes/link3.obj
- link link4: geometry visual mesh filename=../../../robot_models/Panda/newmeshes/link4.obj
- link link5: geometry visual mesh filename=../../../robot_models/Panda/newmeshes/link5.obj
- link link6: geometry visual mesh filename=../../../robot_models/Panda/newmeshes/link6.obj
- link link7: geometry visual mesh filename=../../../robot_models/Panda/newmeshes/link7.obj

File: 05-examples/panda_arm_FT_sensor.urdf (robot description, URDF)
Before this commit: robot panda-sensor, 14 links, 13 joints
Links:
- link link0: geometry visual mesh filename=../../../robot_models/Panda/newmeshes/link0.obj
- link link1: geometry visual mesh filename=../../../robot_models/Panda/newmeshes/link1.obj
- link link2: geometry visual mesh filename=../../../robot_models/Panda/newmeshes/link2.obj
- link link3: geometry visual mesh filename=../../../robot_models/Panda/newmeshes/link3.obj
- link link4: geometry visual mesh filename=../../../robot_models/Panda/newmeshes/link4.obj
- link link5: geometry visual mesh filename=../../../robot_models/Panda/newmeshes/link5.obj
- link link6: geometry visual mesh filename=../../../robot_models/Panda/newmeshes/link6.obj
- link link7: geometry visual mesh filename=../../../robot_models/Panda/newmeshes/link7.obj
